File: Breakout/KiCad/Charge-Seed-Breakout.kicad_sch (KiCad schematic)
At the start: 16 parts, among them U1 JL308-25410G01, U10 JL308-25410G01, U2 JL308-25410G01, U3 P125-1120A0BS116A1, U4 2541FV-20P-B, U5 2541FV-20P-B, U6 P125-1120A0BS116A1, U7 2541FV-20P-B, U8 2541FV-20P-B, U9 JL308-25410G01

Commit message: Exported as v0.1 for production.
Parts:
- removed H1, H2, H3, H4, H5, H6: MountingHole_Pad, clectric-diy:MountingHole_AE, symbol Mechanical:MountingHole_Pad
Other:
- company: clectric.diy -> Copyright © 2025 clectric.diy Licensed under CERN-OHL-S v2
