File: Breakout/KiCad/Charge-Seed-Breakout.kicad_pcb (KiCad board)
At the start: 4 copper layers, 125 x 101 mm, 10 parts, among them U1 JL308-25410G01, U10 JL308-25410G01, U2 JL308-25410G01, U3 P125-1120A0BS116A1, U4 2541FV-20P-B, U5 2541FV-20P-B, U6 P125-1120A0BS116A1, U7 2541FV-20P-B, U8 2541FV-20P-B, U9 JL308-25410G01

Commit message: reducing to 2 layers
Other:
- copper layers 4 -> 2
Changed lines of the file:
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@@
 	(layers
 		(0 "F.Cu" signal "Front")
-		(4 "In1.Cu" signal)
-		(6 "In2.Cu" signal)
 		(2 "B.Cu" signal "Back")
 		(13 "F.Paste" user)
@@
 			(layer "dielectric 1"
 				(type "core")
-				(thickness 0.480066)
+				(thickness 1.510198)
 				(material "FR4")
 				(epsilon_r 4.5)
-				(loss_tangent 0.02)
-			)
-			(layer "In1.Cu"
-				(type "copper")
-				(thickness 0.035)
-			)
-			(layer "dielectric 2"
-				(type "prepreg")
-				(thickness 0.480066)
-				(material "FR4")
-				(epsilon_r 4.5)
-				(loss_tangent 0.02)
-			)
-			(layer "In2.Cu"
-				(type "copper")
-				(thickness 0.035)
-			)
-			(layer "dielectric 3"
-				(type "core")
-				(thickness 0.480066)
-				(material "FR4")
-				(epsilon_r 4.5)
